Commit message: urdf_update

File: urdf/rover.urdf.xacro (robot description, xacro)
@@ -39,4 +39,7 @@
         </inertial>
     </link>
+    <gazebo reference="base_link">
+        <material>Gazebo/Grey</material>
+    </gazebo>
     <joint name="base_joint" type="fixed">
         <parent link="base_footprint"/>
@@ -334,4 +337,7 @@
             </inertial>
         </link>
+        <gazebo reference="front_wheel_link_${prefix}">
+            <material>Gazebo/DarkGrey</material>
+        </gazebo>
         <joint name="front_wheel_joint_${prefix}" type="continuous">
             <parent link="front_wheel_link_${prefix_1}"/>
@@ -369,4 +375,7 @@
             </inertial>
         </link>
+       <gazebo reference="middle_wheel_link_${prefix}">
+            <material>Gazebo/DarkGrey</material>
+        </gazebo>
         <joint name="middle_wheel_joint_${prefix}" type="continuous">
             <parent link="middle_wheel_link_${prefix_1}"/>
@@ -404,4 +413,7 @@
             </inertial>
         </link>
+       <gazebo reference="rear_wheel_link_${prefix}">
+            <material>Gazebo/DarkGrey</material>
+        </gazebo>
         <joint name="rear_wheel_joint_${prefix}" type="continuous">
             <parent link="rear_wheel_link_${prefix_1}"/>
